File: MPPT-Interface-Board.kicad_sch (KiCad schematic)
At the start: 30 parts, among them J1 MPPT A, J2 MPPT X, J3 CarCAN In, J4 CarCAN Out, J5 FUSEBOX, J6 CANDAPTER, Q1 PMV35EPER, U1 RI3-1209S

Commit message: footprints
Parts:
- removed J6: CANDAPTER, DB-9 Connector:AMPHENOL_L77SDE09SA4CH3R, symbol Connector:DE9_Plug_MountingHoles
- C3, C4: footprint (none) -> Capacitor_SMD:C_0805_2012Metric
- JP1: footprint Jumper:SolderJumper-2_P1.3mm_Open_RoundedPad1.0x1.5mm -> Jumper:SolderJumper-2_P1.3mm_Open_TrianglePad1.0x1.5mm
- Q1: symbol utsvt-chips:PMV35EPE -> UTSVT-Chips:PMV35EPE
- TP1, TP2, TP3, TP4, TP5, TP6: footprint (none) -> TestPoint:TestPoint_Pad_1.0x1.0mm
- U1: footprint UTSVT_ICs:RI3_DC_Converter -> UTSVT-ICs:RI3_DC_Converter
- Z1: footprint Zener:BZT52B12QX -> BZT52-B12-QX:BZT52B12QX
Connections:
- no-connect marks 16 -> 8
Other:
- moved on the sheet: J5
