File: MPPT-Interface-Board.kicad_pcb (KiCad board)
At the start: 2 copper layers, 22 parts, among them J1 MPPT CAN 1, J2 MPPT CAN 2, J3 CarCAN 1, J4 CarCAN 2, J5 FUSEBOX, Q1 PMV35EPER, Q2 IRLML0030, U1 ISO6721RBQDRQ1

Commit message: add indicator LEDs
Parts:
- removed D2: SD12_SOD323, Diode_SMD:D_SOD-323
- removed D3: PowerOn, LED_SMD:LED_0805_2012Metric
- removed Q2: IRLML0030, Package_TO_SOT_SMD:SOT-23
- removed R3: 1.5k, Resistor_SMD:R_0805_2012Metric
- removed U1: ISO6721RBQDRQ1, ISO6721R-Q1:SOIC8_D_TEX
- added C5: 10u, Capacitor_SMD:C_0805_2012Metric, F.Cu at (158.6, 86.0)
- C1: value 10u -> 10uF
- J2: footprint Connector_Molex:Molex_Micro-Fit_3.0_43045-0612_2x03_P3.00mm_Vertical -> Connector_Molex:Molex_Micro-Fit_3.0_43650-0215_1x02_P3.00mm_Vertical
Connections:
- C1 pad 1: /Power/+12V_CTRLS_PROT -> +12V
- C1 pad 2: GND -> GNDPWR
- C2 pad 1: +12V -> V_CAN
- C2 pad 2: Net-(Q2-D) -> CGND
- D1 pad 1: GND -> GNDPWR
- D1 pad 2: /Power/+12V_CTRLS -> +12V
- J1 pad 1: +12V -> V_CAN
- J1 pad 2: GNDPWR -> CGND
- J2 pad 1: +12V -> /CAN_H
- J2 pad 2: GNDPWR -> /CAN_L
- J3 pad 2: GND -> CGND
- J4 pad 2: GND -> CGND
- Q1 pad 2: /Power/+12V_CTRLS_PROT -> +12V_PROT
- Q1 pad 3: /Power/+12V_CTRLS -> +12V
- R2 pad 1: GND -> GNDPWR

Commit message: footprints
Parts:
- added C3: 330p, Capacitor_SMD:C_0805_2012Metric, F.Cu at (147.3, 82.5)
- added C4: 470p, Capacitor_SMD:C_0805_2012Metric, F.Cu at (147.3, 85.5)
- added D2: 12V, LED_SMD:LED_0805_2012Metric, F.Cu at (156.2, 76.5)
- added D3: 5V, LED_SMD:LED_0805_2012Metric, F.Cu at (156.2, 79.5)
- added D4: VCAN, LED_SMD:LED_0805_2012Metric, F.Cu at (156.2, 82.6)
- added R3: 5.1k, Resistor_SMD:R_0805_2012Metric, F.Cu at (151.7, 82.4)
- added R4: 1.69k, Resistor_SMD:R_0805_2012Metric, F.Cu at (151.7, 85.3)
- added R5: 3.48k, Resistor_SMD:R_0805_2012Metric, F.Cu at (151.7, 88.3)
- added TP5: VCAN, TestPoint:TestPoint_Pad_1.0x1.0mm, F.Cu at (152.7, 108.5)
- added TP6: CGND, TestPoint:TestPoint_Pad_1.0x1.0mm, F.Cu at (152.7, 111.6)
- added U1: RI3-1209S, UTSVT-ICs:RI3_DC_Converter, F.Cu at (151.6, 97.1)
- added Z1: BZT52-B12-QX, BZT52-B12-QX:BZT52B12QX, F.Cu at (148.7, 115.5)
- C1, C2: value 10uF -> 10u
- J1: value MPPT CAN 1 -> MPPT A
- J2: value MPPT CAN 2 -> MPPT X; footprint Connector_Molex:Molex_Micro-Fit_3.0_43650-0215_1x02_P3.00mm_Vertical -> Connector_Molex:Molex_Micro-Fit_3.0_43045-0612_2x03_P3.00mm_Vertical
- J3: value CarCAN 1 -> CarCAN In
- J4: value CarCAN 2 -> CarCAN Out
- JP1: footprint Jumper:SolderJumper-2_P1.3mm_Open_RoundedPad1.0x1.5mm -> Jumper:SolderJumper-2_P1.3mm_Open_TrianglePad1.0x1.5mm
- TP1: value 12V_UNISO -> CGND; footprint TestPoint:TestPoint_Keystone_5005-5009_Compact -> TestPoint:TestPoint_Pad_1.0x1.0mm
- TP2: value GND_UNISO -> GNDPWR; footprint TestPoint:TestPoint_Keystone_5005-5009_Compact -> TestPoint:TestPoint_Pad_1.0x1.0mm
- TP3: value +5V_TP -> 5V; footprint TestPoint:TestPoint_Keystone_5005-5009_Compact -> TestPoint:TestPoint_Pad_1.0x1.0mm
- TP4: value GND_TP -> 12V; footprint TestPoint:TestPoint_Keystone_5005-5009_Compact -> TestPoint:TestPoint_Pad_1.0x1.0mm
- moved Q1 46.1 mm to (154.8, 115.5)
- moved D1 39.9 mm to (156.4, 108.5)
- moved TP1 38.9 mm to (146.6, 108.5)
- moved TP2 36.9 mm to (146.6, 111.6)
- moved J5 35.0 mm to (149.4, 102.7)
- moved TP3 28.9 mm to (149.7, 108.5)
- moved TP4 26.9 mm to (149.7, 111.6)
- moved G*** 25.2 mm to (126.8, 99.8), turned to 90 degrees
- moved JP1 23.7 mm to (156.1, 85.9)
- moved R1 18.5 mm to (151.7, 76.5)
- moved J2 16.1 mm to (134.5, 89.3)
- moved J3 16.1 mm to (134.5, 100.1)
- moved J4 16.1 mm to (134.5, 111.0)
- moved J1 16.1 mm to (134.5, 78.5)
- moved C5 11.5 mm to (147.3, 88.5)
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Connections:
- C1 pad 1: +12V -> +12V_PROT
- J2 pad 1: /CAN_H -> V_CAN
- J2 pad 2: /CAN_L -> CGND2
- J4 pad 2: CGND -> CGND2
- J4 pad 4: /CAN_H -> /CAN_H2
- J4 pad 5: /CAN_L -> /CAN_L2
- TP1 pad 1: +12V -> CGND
- TP4 pad 1: GND -> +12V_PROT

Commit message: initial layout (unrouted)
Parts:
- added H1: MountingHole, MountingHole:MountingHole_3mm, F.Cu at (99.0, 65.8)
- added H2: MountingHole, MountingHole:MountingHole_3mm, F.Cu at (134.2, 65.8)
- added H3: MountingHole, MountingHole:MountingHole_3mm, F.Cu at (134.2, 103.8)
- added H4: MountingHole, MountingHole:MountingHole_3mm, F.Cu at (99.0, 103.8)
- C1, C2, C3, C4, C5, D1, JP1, Q1, R1, R2, R3, R4, R5, Z1: moved to B.Cu
- TP6: value CGND -> CGND2
- moved TP5 68.0 mm to (94.0, 74.2)
- moved TP6 61.1 mm to (94.0, 94.5)
- moved D1 57.2 mm to (104.0, 85.5)
- moved Q1 56.7 mm to (107.5, 84.3), turned to -90 degrees
- moved Z1 54.1 mm to (107.6, 80.2), turned to 180 degrees
- moved J5 51.9 mm to (100.2, 86.2), turned to 90 degrees
- moved R2 48.1 mm to (103.8, 83.2)
- moved TP2 45.5 mm to (107.5, 88.2)
- moved TP3 42.3 mm to (107.5, 112.0)
- moved JP1 40.9 mm to (117.8, 100.0), turned to 180 degrees
- moved D2 40.5 mm to (115.8, 78.5)
- moved R1 39.9 mm to (117.8, 97.5), turned to 180 degrees
- moved C5 37.0 mm to (110.5, 84.5), turned to -90 degrees
- moved U1 35.4 mm to (117.5, 87.8)
- moved R3 35.2 mm to (116.5, 82.5), turned to 90 degrees
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Connections:
- C4 pad 1: +12V -> +12V_PROT
- JP1 pad 2: /CAN_L -> /CAN_L2
- R1 pad 2: /CAN_H -> /CAN_H2
- TP6 pad 1: CGND -> CGND2
Routing:
- added copper zone on B.Cu, net +5V
- added copper zone on F.Cu, net CGND
- added copper zone on F.Cu, net CGND2
- added copper zone on B.Cu, net GNDPWR
- added copper zone on B.Cu, net V_CAN
Other:
- board outline added: 41.8 x 44.5 mm
- board text added: "TODO: silks for connectors H,L,+-"

Commit message: add silk labels
Parts:
- moved TP2 15.2 mm to (92.8, 84.5)
- moved D2 8.46 mm to (108.8, 83.2)
- moved R3 4.83 mm to (112.0, 80.8)
- moved J1 1.25 mm to (121.2, 71.5)
- moved J2 1.25 mm to (106.0, 71.5)
Other:
- board text added: "5V"
- board text added: "CGND"
- board text added: "CGND2"
- board text added: "H L"
- board text added: "H2 L2"
- board text added: "L H"
- board text added: "L2 H2"
- board text added: "TODO: silks for connectors H,L,+- and others :D"
- board text added: "VCAN"
- board text removed: "TODO: silks for connectors H,L,+-"
Changed lines of the file:
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@@
 	(footprint "Connector_Molex:Molex_Micro-Fit_3.0_43045-0612_2x03_P3.00mm_Vertical"
 		(layer "F.Cu")
-		(at 121.25 70.25)
+		(at 121.25 71.5)
 		(descr "Molex Micro-Fit 3.0 Connector System, 43045-0612 (compatible alternatives: 43045-0613, 43045-0624), 3 Pins per row (http://www.molex.com/pdm_docs/sd/430450212_sd.pdf), generated with kicad-footprint-generator")
 		(tags "connector Molex Micro-Fit_3.0 vertical")
 		(property "Reference" "J1"
-			(at 3 -3.67 0)
+			(at -3 -3.5 0)
 			(layer "F.SilkS")
 			(effects
@@
 		)
 		(property "Value" "MPPT A"
-			(at 3 7.51 0)
+			(at 3 7.5 0)
 			(layer "F.SilkS" knockout)
 			(effects
@@
 		(tags "connector Molex Micro-Fit_3.0 vertical")
 		(property "Reference" "J3"
-			(at 3 -3.67 360)
+			(at 9 -3.67 360)
 			(layer "F.SilkS")
 			(effects
@@
 		(tags "connector Molex Micro-Fit_3.0 vertical")
 		(property "Reference" "J4"
-			(at 3 -3.67 360)
+			(at 9 -3.67 360)
 			(layer "F.SilkS")
 			(effects
@@
 		)
 		(property "Value" "CarCAN Out"
-			(at 3 7.51 0)
+			(at 3 7.5 0)
 			(layer "F.SilkS" knockout)
 			(effects
@@
 	(footprint "LED_SMD:LED_0805_2012Metric"
 		(layer "F.Cu")
-		(at 115.75 78.5)
+		(at 108.75 83.25)
 		(descr "LED SMD 0805 (2012 Metric), square (rectangular) end terminal, IPC_7351 nominal, (Body size source: https://docs.google.com/spreadsheets/d/1BsfQQcO9C6DZCsRaXUlFlo91Tg2WpOkGARC1WS5S8t0/edit?usp=sharing), generated with kicad-footprint-generator")
 		(tags "LED")
@@
 		)
 		(property "Value" "12V"
-			(at 0 1.65 0)
+			(at 0 -1.75 0)
 			(layer "F.SilkS" knockout)
 			(effects
@@
 	(footprint "Connector_Molex:Molex_Micro-Fit_3.0_43045-0612_2x03_P3.00mm_Vertical"
 		(layer "F.Cu")
-		(at 106 70.25)
+		(at 106 71.5)
 		(descr "Molex Micro-Fit 3.0 Connector System, 43045-0612 (compatible alternatives: 43045-0613, 43045-0624), 3 Pins per row (http://www.molex.com/pdm_docs/sd/430450212_sd.pdf), generated with kicad-footprint-generator")
 		(tags "connector Molex Micro-Fit_3.0 vertical")
 		(property "Reference" "J2"
-			(at 3 -3.67 0)
+			(at -3 -3.5 0)
 			(layer "F.SilkS")
 			(effects
@@
 		)
 		(property "Value" "MPPT X"
-			(at 3 7.51 0)
+			(at 3 7.5 0)
 			(layer "F.SilkS" knockout)
 			(effects
@@
 	(footprint "TestPoint:TestPoint_Pad_1.0x1.0mm"
 		(layer "F.Cu")
-		(at 107.5 88.25)
+		(at 92.75 84.5)
 		(descr "SMD rectangular pad as test Point, square 1.0mm side length")
 		(tags "test point SMD pad rectangle square")
@@
 	(footprint "Resistor_SMD:R_0805_2012Metric"
 		(layer "B.Cu")
-		(at 116.5 82.5 90)
+		(at 112 80.75 90)
 		(descr "Resistor SMD 0805 (2012 Metric), square (rectangular) end terminal, IPC_7351 nominal, (Body size source: IPC-SM-782 page 72, https://www.pcb-3d.com/wordpress/wp-content/uploads/ipc-sm-782a_amendment_1_and_2.pdf), generated with kicad-footprint-generator")
 		(tags "resistor")
@@
 		(layer "Edge.Cuts")
 	)
-	(gr_text "TODO: silks for connectors H,L,+-"
+	(gr_text "CGND2"
+		(at 109.5 106.25 90)
+		(layer "F.SilkS" knockout)
+		(effects
+			(font
+				(size 0.8 0.8)
+				(thickness 0.12)
+			)
+			(justify left bottom)
+		)
+	)
+	(gr_text "L2  H2"
+		(at 107.75 94 0)
+		(layer "F.SilkS")
+		(effects
+			(font
+				(size 1 1)
+				(thickness 0.15)
+			)
+			(justify left bottom)
+		)
+	)
+	(gr_text "H   L"
+		(at 120.75 78 0)
+		(layer "F.SilkS")
+		(effects
+			(font
+				(size 1 1)
+				(thickness 0.15)
+			)
+			(justify left bottom)
+		)
+	)
+	(gr_text "VCAN"
+		(at 121.75 68.5 90)
+		(layer "F.SilkS" knockout)
+		(effects
+			(font
+				(size 0.8 0.8)
+				(thickness 0.12)
+			)
+			(justify left bottom)
+		)
+	)
+	(gr_text "5V"
+		(at 127.75 103.75 90)
+		(layer "F.SilkS" knockout)
+		(effects
+			(font
+				(size 0.8 0.8)
+				(thickness 0.12)
+			)
+			(justify left bottom)
+		)
+	)
+	(gr_text "CGND2"
+		(at 109.5 68.5 90)
+		(layer "F.SilkS" knockout)
+		(effects
+			(font
+				(size 0.8 0.8)
+				(thickness 0.12)
+			)
+			(justify left bottom)
+		)
+	)
+	(gr_text "L   H"
+		(at 123.75 94 0)
+		(layer "F.SilkS")
+		(effects
+			(font
+				(size 1 1)
+				(thickness 0.15)
+			)
+			(justify left bottom)
+		)
+	)
+	(gr_text "CGND"
+		(at 124.75 105.5 90)
+		(layer "F.SilkS" knockout)
+		(effects
+			(font
+				(size 0.8 0.8)
+				(thickness 0.12)
+			)
+			(justify left bottom)
+		)
+	)
+	(gr_text "CGND"
+		(at 124.75 68.5 90)
+		(layer "F.SilkS" knockout)
+		(effects
+			(font
+				(size 0.8 0.8)
+				(thickness 0.12)
+			)
+			(justify left bottom)
+		)
+	)
+	(gr_text "5V"
+		(at 112.5 103.75 90)
+		(layer "F.SilkS" knockout)
+		(effects
+			(font
+				(size 0.8 0.8)
+				(thickness 0.12)
+			)
+			(justify left bottom)
+		)
+	)
+	(gr_text "H2  L2"
+		(at 104.75 78 0)
+		(layer "F.SilkS")
+		(effects
+			(font
+				(size 1 1)
+				(thickness 0.15)
+			)
+			(justify left bottom)
+		)
+	)
+	(gr_text "VCAN"
+		(at 106.5 68.5 90)
+		(layer "F.SilkS" knockout)
+		(effects
+			(font
+				(size 0.8 0.8)
+				(thickness 0.12)
+			)
+			(justify left bottom)
+		)
+	)
+	(gr_text "TODO: silks for connectors H,L,+- and others :D"
 		(at 99.5 58.25 0)
 		(layer "Cmts.User")

Commit message: routed
Parts:
- TP2, TP4: moved to B.Cu
- moved TP2 40.5 mm to (133.2, 84.8), turned to 180 degrees
- moved TP4 27.0 mm to (116.8, 82.8), turned to 180 degrees
- moved TP5 22.2 mm to (113.8, 64.2)
- moved TP3 10.1 mm to (114.2, 104.4)
- moved TP1 6.38 mm to (134.2, 97.4)
- moved TP6 5.78 mm to (99.0, 97.4)
- moved D1 0.90 mm to (104.5, 86.2), turned to 90 degrees
- moved D2 0.75 mm to (109.5, 83.2)
- moved G*** 0.25 mm to (134.2, 84.8)
Routing:
- net /CAN_L2: track 0.00 -> 40.9 mm, vias 0 -> 1
- net /CAN_H2: track 0.00 -> 32.9 mm, vias 0 -> 1
- net /CAN_H: track 0.00 -> 28.8 mm, vias 0 -> 1
- net /CAN_L: track 0.00 -> 21.8 mm, vias 0 -> 1
- net Net-(D4-A): track 0.00 -> 8.58 mm, vias 0 -> 1
- net Net-(D3-A): track 0.00 -> 6.59 mm, vias 0 -> 1
- net CGND: track 0.00 -> 5.34 mm
- net Net-(D2-A): track 0.00 -> 4.70 mm, vias 0 -> 1
- net GNDPWR: track 0.00 -> 3.43 mm, vias 0 -> 1
- net Net-(JP1-A): track 0.00 -> 2.60 mm
- net +5V: track 0.00 -> 1.93 mm, vias 0 -> 1
- net V_CAN: track 0.00 -> 1.60 mm, vias 0 -> 1
- added copper zone on B.Cu, net +12V
- added copper zone on B.Cu, net +12V_PROT
- added copper zone on B.Cu, net Net-(Q1-G)
Other:
- board text added: "+ -"

Commit message: redo layout/routing/silks
Parts:
- added G***: LOGO, LOGO, F.Cu at (99.0, 73.0)
- added G***: LOGO, LOGO, B.Cu at (126.8, 102.0)
- added JP2: CAN START, Jumper:SolderJumper-2_P1.3mm_Open_TrianglePad1.0x1.5mm, B.Cu at (116.9, 67.0)
- added LOGO1: UTSVT Logo, UTSVT-Special:UTSVT_Logo_Symbol, B.Cu at (127.0, 84.2)
- added R6: 120, Resistor_SMD:R_0805_2012Metric, B.Cu at (116.9, 69.5)
- J3, J4: footprint Connector_Molex:Molex_Micro-Fit_3.0_43045-0612_2x03_P3.00mm_Vertical -> UTSVT-Connectors:Molex_MicroFit3.0_1x4xP3.00mm_PolarizingPeg_Vertical
- JP1: value CAN TERM -> CAN END
- moved TP6 8.08 mm to (104.0, 103.8)
- moved TP1 8.04 mm to (130.0, 104.2)
- moved J3 5.43 mm to (131.6, 96.0)
- moved J4 3.50 mm to (110.6, 96.0)
- moved JP1 2.56 mm to (116.9, 102.4)
- moved R1 2.56 mm to (116.9, 99.9)
- moved H3 1.75 mm to (134.2, 102.0)
- moved H4 1.75 mm to (99.0, 102.0)
- moved R4 1.65 mm to (134.4, 93.2)
- moved TP3 0.60 mm to (114.2, 103.8)
Connections:
- J3 pad 3: unconnected-(J3-Pin_3-Pad3) -> /CAN_H
- J3 pad 4: /CAN_H -> /CAN_L
- J4 pad 3: unconnected-(J4-Pin_3-Pad3) -> /CAN_H2
- J4 pad 4: /CAN_H2 -> /CAN_L2
Routing:
- net /CAN_L: track 21.8 -> 38.4 mm, vias 1 -> 2
- net /CAN_H: track 28.8 -> 36.3 mm, vias 1 -> 2
- net /CAN_L2: track 40.9 -> 47.8 mm, vias 1 -> 2
- net /CAN_H2: track 32.9 -> 38.4 mm, vias 1 -> 2
- net Net-(JP2-A): track 0.00 -> 2.58 mm
- net Net-(D3-A): track 6.59 -> 7.17 mm
Other:
- board text added: "Grid size is 0.25mm"
- board text added: "H"
- board text added: "H2"
- board text added: "L"
- board text added: "L2"
- board text added: "Ravi Shah 2025"
- board text removed: "L H"
- board text removed: "L2 H2"

Commit message: lil smaller
Parts:
- moved TP1 5.84 mm to (124.2, 103.2)
- moved TP3 3.00 mm to (111.5, 102.5)
- moved TP6 1.27 mm to (104.2, 102.5)
- moved JP1 1.15 mm to (116.9, 101.2)
- moved R1 1.15 mm to (116.9, 98.8)
- moved G*** 1.00 mm to (126.8, 101.0)
Routing:
- net /CAN_H2: track 38.4 -> 39.5 mm
Other:
- board size 41.8 x 44.5 mm -> 41.8 x 42.8 mm
- board text removed: "TODO: silks for connectors H,L,+- and others :D"
